File: ohm3/hw/simple_mesh/simple_mesh.kicad_pcb (KiCad board)
At the start: 2 copper layers, 25.4 x 54.6 mm, 21 parts, among them IC1 RaspberryPi_Pico, IC2 SX1262, J3 Conn_01x04, J4 Conn_01x04

Commit message: BUG - need to connect BUSY to DI02
Parts:
- D4: footprint Diode_SMD:D_SOD-123F -> Diode_SMD:D_SMA
Connections:
- IC1 pad 4: LORA_DIO2 -> LORA_BUSY
- IC2 pad 5: LORA_DIO2 -> unconnected-(IC2-DIO2-Pad5)
- IC2 pad 9: unconnected-(IC2-BUSY-Pad9) -> LORA_BUSY
Routing:
- net LORA_DIO2: track 51.1 -> 0.00 mm, vias 3 -> 0
- net LORA_BUSY: track 0.00 -> 48.8 mm, vias 0 -> 1
Other:
- board text added: "v0.2"
